Commit message: Added joint limits

File: bexter_combined_urdf/urdf/bexter_combined_urdf.urdf (robot description, URDF)
Before this commit: robot bexter_combined_urdf, 5 links, 4 joints
Joints:
- joint joint_1: limit lower=0 upper=0 effort=1.4 velocity=0.9 -> lower=-1.57 upper=1.57 effort=1.4 velocity=0.9; type continuous -> revolute
- joint joint_3: limit lower=0 upper=0 effort=1.4 velocity=0.9 -> lower=-3.14 upper=1.57 effort=1.4 velocity=0.9; type continuous -> revolute

Commit message: Adding bexter launch and motor fixes for correction action while loop and prevent large motor jumps

File: bexter_combined_urdf/urdf/bexter_combined_urdf.urdf (robot description, URDF)
Before this commit: robot bexter_combined_urdf, 5 links, 4 joints
Joints:
- joint joint_1: limit lower=-1.57 upper=1.57 effort=1.4 velocity=0.9 -> lower=-1.57 upper=1.57 effort=1.4 velocity=3.14
- joint joint_2: limit lower=0 upper=0 effort=1.4 velocity=0.9 -> lower=0 upper=0 effort=1.4 velocity=3.14
- joint joint_3: limit lower=-3.14 upper=1.57 effort=1.4 velocity=0.9 -> lower=-3.14 upper=1.57 effort=1.4 velocity=3.14
