Commit message: Adding new motion planning with updated model

File: bexter_urdf_final_combined/urdf/bexter_urdf_final_combined.urdf (robot description, URDF)
Before this commit: robot bexter_urdf_final_combined, 5 links, 4 joints
Links:
- link base_link: geometry collision mesh filename=package://bexter_urdf_final_combined/meshes/base_link_colli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; visual mesh filename=package://bexter_urdf_final_combined/meshes/base_link.STL
- link end_effector: geometry collision mesh filename=package://bexter_urdf_final_combined/meshes/end_effector_co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; visual mesh filename=package://bexter_urdf_final_combined/meshes/end_effector.STL
- link link_0: geometry collision mesh filename=package://bexter_urdf_final_combined/meshes/link_0_collisio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; visual mesh filename=package://bexter_urdf_final_combined/meshes/link_0.STL
- link link_1: geometry collision mesh filename=package://bexter_urdf_final_combined/meshes/link_1_collisio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; visual mesh filename=package://bexter_urdf_final_combined/meshes/link_1.STL
- link link_2: geometry collision mesh filename=package://bexter_urdf_final_combined/meshes/link_2_collisio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; visual mesh filename=package://bexter_urdf_final_combined/meshes/link_2.STL
Joints:
- joint joint_1: limit lower=-1.57 upper=1.57 effort=1.4 velocity=3.14 -> lower=-1.57 upper=1.57 effort=1.4 velocity=2.0; type continuous -> revolute
- joint joint_2: limit lower=0 upper=0 effort=1.4 velocity=3.14 -> lower=-1.57 upper=1.57 effort=1.4 velocity=2.0
- joint joint_3: limit lower=-3.14 upper=1.57 effort=1.4 velocity=3.14 -> lower=-1.57 upper=1.57 effort=1.4 velocity=2.0
